File: TouchPanelPrototype.sch (EAGLE design)
At the start: 32 parts, among them IC1 AT42QT1040, IC2 MCP1700T-3302, J1 Interface

Commit message: foo
Other:
- note removed: "Worldwide grid voltage compatible: 90-260 VAC 50-60 Hz."
Changed lines of the file:
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@@
 <text x="22.86" y="269.24" size="1.4224" layer="91"></text>
 <text x="22.86" y="266.7" size="1.4224" layer="91"></text>
-<text x="5.08" y="7.62" size="1.778" layer="98" ratio="16">Worldwide grid voltage compatible: 90-260 VAC 50-60 Hz.</text>
 <text x="68.834" y="185.42" size="1.27" layer="98"></text>
 <text x="162.56" y="144.78" size="1.27" layer="98"></text>
